Commit message: backup tmp xacro

File: arm_description/urdf/arm.xacro (robot description, xacro)
@@ -3,5 +3,5 @@
 <robot name="arm" xmlns:xacro="http://ros.org/wiki/xacro">
   <!-- ======================== GLOBAL CONSTANTS ======================== -->
-  <xacro:property name="M_PI" value="3.14159" />
+  <xacro:property name="M_PI" value="3.141592653589793" />
   <xacro:property name="COLLISION_SCALE" value="0.80" />
   <!-- ======================== MATERIAL DEFINITIONS ======================== -->

File: arm_description/urdf/lekiwi_arm.xacro (robot description, xacro)
@@ -2,5 +2,5 @@
 <robot name="LeKiwi_Arm" xmlns:xacro="http://ros.org/wiki/xacro">
   <!-- ======================== GLOBAL CONSTANTS ======================== -->
-  <xacro:property name="M_PI" value="3.14159" />
+  <xacro:property name="M_PI" value="3.141592653589793" />
   <!-- ======================== MATERIAL DEFINITIONS ======================== -->
   <material name="Black">
@@ -465,5 +465,5 @@
     child="SO_ARM100_08k_116_Square-v1"
     xyz="0.0346 0.010249999999999987 -0.032799999999999975"
-    rpy="3.141592653589793 1.7181275903033976e-32 -3.1373434374976504e-48"
+    rpy="1.5707963267948966 1.7181275903033976e-32 -3.1373434374976504e-48"
     axis="1.0 0.0 0.0" />
   <xacro:continuous_joint name="joint3"
@@ -471,5 +471,5 @@
     child="SO_ARM100_08k_Mirror-v1"
     xyz="0.0346 -0.013069710000000002 0.03178184000000002"
-    rpy="-6.842277657836021e-49 -3.4512664603419266e-31 -1.3877787807814457e-17"
+    rpy="${M_PI} -3.4512664603419266e-31 -1.3877787807814457e-17"
     axis="1.0 0.0 0.0" />
   <xacro:continuous_joint name="joint4"
@@ -477,5 +477,5 @@
     child="Wrist_Roll_Pitch_08i-v1"
     xyz="0.0346 -0.03408158 0.004398620000000015"
-    rpy="3.1415926535897922 9.860761315262648e-32 -9.503163413661107e-47"
+    rpy="${M_PI*1.5} 9.860761315262648e-32 -9.503163413661107e-47"
     axis="1.0 0.0 9.860761315262648e-32" />
   <xacro:continuous_joint name="joint5"
