Commit message: update arm xaceo for lekiwi

File: arm_description/urdf/lekiwi_arm.xacro (robot description, xacro)
@@ -1,4 +1,6 @@
 <?xml version="1.0"?>
 <robot name="LeKiwi_Arm" xmlns:xacro="http://ros.org/wiki/xacro">
+  <!-- ======================== GLOBAL CONSTANTS ======================== -->
+  <xacro:property name="M_PI" value="3.14159" />
   <!-- ======================== MATERIAL DEFINITIONS ======================== -->
   <material name="Black">
@@ -104,8 +106,8 @@
     iyz="0.00024876935781550404"
     ixz="-1.4799628966957228e-07"
-    visual_xyz="-0.039999997308103726 -0.058051990747593187 -0.0024000000000000644"
-    visual_rpy="1.5707963267948968 6.378522481755146e-34 -3.141592653589793"
-    collision_xyz="-0.039999997308103726 -0.058051990747593187 -0.0024000000000000644"
-    collision_rpy="1.5707963267948968 6.378522481755146e-34 -3.141592653589793" />
+    visual_xyz="-0.058051990747593187 0.039999997308103726 -0.0024000000000000644"
+    visual_rpy="1.5707963267948968 6.378522481755146e-34 -4.712388980384690"
+    collision_xyz="-0.058051990747593187 0.039999997308103726 -0.0024000000000000644"
+    collision_rpy="1.5707963267948968 6.378522481755146e-34 -4.712388980384690" />
   <!-- ======================== STRUCTURAL LINKS ======================== -->
   <!-- WaveShare Mounting Plate -->
@@ -386,11 +388,11 @@
     parent="base_link"
     child="WaveShare_Mounting_Plate_01d-v1"
-    xyz="-0.04 -0.07525199 0.060300000000000006"
-    rpy="3.141592653589793 6.259293778842913e-51 2.356194490192345" />
+    xyz="-0.07525199 0.04 0.060300000000000006"
+    rpy="3.141592653589793 6.259293778842913e-51 0.7853981633974485" />
   <xacro:fixed_joint name="Base_08q-v1_Rigid-44"
     parent="base_link"
     child="STS3215_03a-v1"
-    xyz="-0.029750000000000002 -0.045651989999999996 0.027800000000000002"
-    rpy="1.5707963267948966 -8.851978152917189e-51 -2.4803256509655576e-48" />
+    xyz="-0.045651989999999996 0.029750000000000002 0.027800000000000002"
+    rpy="1.5707963267948966 -8.851978152917189e-51 -1.5707963267948966" />
   <xacro:fixed_joint name="Rotation_Pitch_08i-v1_Rigid-46"
     parent="Rotation_Pitch_08i-v1"
@@ -401,6 +403,6 @@
     parent="base_link"
     child="Passive_Horn_01-v1"
-    xyz="-0.04 -0.012851990000000004 0.013599999999999994"
-    rpy="-1.5707963267948966 -8.851978152917189e-51 -2.4803256509655576e-48" />
+    xyz="-0.012851990000000004 0.04 0.013599999999999994"
+    rpy="-1.5707963267948966 -8.851978152917189e-51 -1.5707963267948966" />
   <xacro:fixed_joint name="Rotation_Pitch_08i-v1_Rigid-48"
     parent="Rotation_Pitch_08i-v1"

Commit message: forword front x for base link

File: arm_description/urdf/lekiwi_arm.xacro (robot description, xacro)
@@ -12,4 +12,7 @@
   <material name="Blue">
     <color rgba="0 0 1 1" />
+  </material>
+  <material name="Gray">
+    <color rgba="0.5 0.5 0.5 1" />
   </material>
   <!-- ======================== XACRO PROPERTIES ======================== -->
@@ -45,4 +48,5 @@
           <mesh filename="${mesh_prefix}/${mesh_file}" scale="${mesh_scale}" />
         </geometry>
+        <material name="Gray" />
       </visual>
       <collision name="${name}_collision">
@@ -89,4 +93,8 @@
     <xacro:inertial_matrix mass="500" />
   </link>
+  <!-- Base Link with origin at joint1 axis (virtual link) -->
+  <link name="base_link">
+    <xacro:inertial_matrix mass="0.001" />
+  </link>
   <xacro:fixed_joint name="bottom_joint"
     parent="base_link"
@@ -94,6 +102,6 @@
     xyz="0.0 0.0 0.0"
     rpy="0.0 0.0 0.0" />
-  <!-- Base Link (机械臂底座) -->
-  <xacro:mesh_link name="base_link"
+  <!-- Physical base link (renamed to base_link_physical) -->
+  <xacro:mesh_link name="base_link_physical"
     mesh_file="Base_08q-v1.stl"
     inertial_xyz="-0.03999704723368316 -0.03974905501648025 0.021865523723532104"
@@ -110,4 +118,10 @@
     collision_xyz="-0.058051990747593187 0.039999997308103726 -0.0024000000000000644"
     collision_rpy="1.5707963267948968 6.378522481755146e-34 -4.712388980384690" />
+  <!-- Connect base_link to base_link_physical with offset to joint1 axis -->
+  <xacro:fixed_joint name="base_to_physical"
+    parent="base_link"
+    child="base_link_physical"
+    xyz="0.012852 -0.04000 0.0"
+    rpy="0.0 0.0 0.0" />
   <!-- ======================== STRUCTURAL LINKS ======================== -->
   <!-- WaveShare Mounting Plate -->
@@ -386,10 +400,10 @@
   <!-- Fixed Joints -->
   <xacro:fixed_joint name="Base_08q-v1_Rigid-43"
-    parent="base_link"
+    parent="base_link_physical"
     child="WaveShare_Mounting_Plate_01d-v1"
     xyz="-0.07525199 0.04 0.060300000000000006"
     rpy="3.141592653589793 6.259293778842913e-51 0.7853981633974485" />
   <xacro:fixed_joint name="Base_08q-v1_Rigid-44"
-    parent="base_link"
+    parent="base_link_physical"
     child="STS3215_03a-v1"
     xyz="-0.045651989999999996 0.029750000000000002 0.027800000000000002"
@@ -401,5 +415,5 @@
     rpy="-3.944304526105059e-31 -4.116117285135399e-31 -2.781046729970605e-32" />
   <xacro:fixed_joint name="Base_08q-v1_Rigid-47"
-    parent="base_link"
+    parent="base_link_physical"
     child="Passive_Horn_01-v1"
     xyz="-0.012851990000000004 0.04 0.013599999999999994"

Commit message: commit complet lekiwi arm xacro

File: arm_description/urdf/lekiwi_arm.xacro (robot description, xacro)
@@ -73,4 +73,14 @@
       <child link="${child}" />
       <axis xyz="${axis}" />
+    </joint>
+  </xacro:macro>
+  <!-- Macro for creating a revolute joint -->
+  <xacro:macro name="revolute_joint" params="name parent child xyz rpy axis lower upper effort velocity">
+    <joint name="${name}" type="revolute">
+      <origin xyz="${xyz}" rpy="${rpy}" />
+      <parent link="${parent}" />
+      <child link="${child}" />
+      <axis xyz="${axis}" />
+      <limit lower="${lower}" upper="${upper}" effort="${effort}" velocity="${velocity}" />
     </joint>
   </xacro:macro>
@@ -455,39 +465,46 @@
     rpy="1.5707963267948966 -0.0 2.181661564992912" />
   <!-- Continuous Joints (Actuated) -->
-  <xacro:continuous_joint name="joint1"
+  <xacro:revolute_joint name="joint1"
     parent="STS3215_03a-v1"
     child="Rotation_Pitch_08i-v1"
     xyz="-0.010250000000000084 0.03459999999999999 -0.032799999999999996"
     rpy="1.5707963267948966 -2.781046729970605e-32 3.94430452610506e-31"
-    axis="-3.944304526105059e-31 3.944304526105059e-31 1.0" />
-  <xacro:continuous_joint name="joint2"
+    axis="-3.944304526105059e-31 3.944304526105059e-31 1.0"
+    lower="-2.96" upper="2.96" effort="300" velocity="1" />
+  <xacro:revolute_joint name="joint2"
     parent="STS3215_03a-v1-1"
     child="SO_ARM100_08k_116_Square-v1"
     xyz="0.0346 0.010249999999999987 -0.032799999999999975"
     rpy="1.5707963267948966 1.7181275903033976e-32 -3.1373434374976504e-48"
-    axis="1.0 0.0 0.0" />
-  <xacro:continuous_joint name="joint3"
+    axis="1.0 0.0 0.0"
+    lower="-2.35" upper="2.35" effort="300" velocity="1" />
+  <xacro:revolute_joint name="joint3"
     parent="STS3215_03a-v1-2"
     child="SO_ARM100_08k_Mirror-v1"
     xyz="0.0346 -0.013069710000000002 0.03178184000000002"
     rpy="${M_PI} -3.4512664603419266e-31 -1.3877787807814457e-17"
-    axis="1.0 0.0 0.0" />
-  <xacro:continuous_joint name="joint4"
+    axis="1.0 0.0 0.0"
+    lower="-3.14" upper="0" effort="300" velocity="1" />
+  <xacro:revolute_joint name="joint4"
     parent="STS3215_03a-v1-3"
     child="Wrist_Roll_Pitch_08i-v1"
     xyz="0.0346 -0.03408158 0.004398620000000015"
     rpy="${M_PI*1.5} 9.860761315262648e-32 -9.503163413661107e-47"
-    axis="1.0 0.0 9.860761315262648e-32" />
-  <xacro:continuous_joint name="joint5"
+    axis="1.0 0.0 9.860761315262648e-32"
+    lower="-2.14" upper="1.57" effort="300" velocity="1" />
+  <xacro:revolute_joint name="joint5"
     parent="STS3215_03a_Wrist_Roll-v1"
     child="Wrist_Roll_08c-v1"
     xyz="-0.028999999999999998 0.00810632 0.006869499999999995"
     rpy="3.141592653589793 -0.0 0.0"
-    axis="0.0 0.42261799999999994 -0.9063079999999999" />
-  <xacro:continuous_joint name="finger_joint1"
+    axis="0.0 0.42261799999999994 -0.9063079999999999"
+    lower="-3.14" upper="3.14" effort="300" velocity="1" />
+  <!-- rpy="-1.5707963267948968 3.944304526105059e-31 -1.9721522630525295e-31" -->
+  <xacro:revolute_joint name="finger_joint1"
     parent="STS3215_03a-v1-4"
     child="Moving_Jaw_08d-v1"
     xyz="-0.032799999999999996 -0.023912249999999986 0.027026410000000018"
-    rpy="-1.5707963267948968 3.944304526105059e-31 -1.9721522630525295e-31"
-    axis="-2.74128770133849e-31 -0.9063079999999999 -0.422618" />
+    rpy="-2.007130025415877483 0.436331985775628373 -1.570800379727681273"
+    axis="2.74128770133849e-31 0.9063079999999999 0.422618"
+    lower="-1.5708" upper="0" effort="100" velocity="1.0" />
 </robot>

Commit message: add grasp frame and camera frame

File: arm_description/urdf/lekiwi_arm.xacro (robot description, xacro)
@@ -1,4 +1,4 @@
 <?xml version="1.0"?>
-<robot name="LeKiwi_Arm" xmlns:xacro="http://ros.org/wiki/xacro">
+<robot name="lekiwi_arm" xmlns:xacro="http://ros.org/wiki/xacro">
   <!-- ======================== GLOBAL CONSTANTS ======================== -->
   <xacro:property name="M_PI" value="3.141592653589793" />
@@ -407,4 +407,8 @@
     collision_xyz="0.0060386479186058575 -0.01378730883655603 -0.012862534163259838"
     collision_rpy="-0.17453292519943064 -0.9599310885968775 -3.141592653589793" />
+  <!-- Camera frame Model -->
+  <link name="camera_optical_frame" />
+   <!-- ======================== END EFFECTOR ======================== -->
+  <link name="grasping_frame" />
   <!-- ======================== JOINTS ======================== -->
   <!-- Fixed Joints -->
@@ -464,4 +468,15 @@
     xyz="0.0015500000000000004 0.00712333000000001 0.06397354"
     rpy="1.5707963267948966 -0.0 2.181661564992912" />
+   <xacro:fixed_joint name="camera_optical_joint"
+    parent="Camera-Model-v3-1"
+    child="camera_optical_frame"
+    xyz="0 0 0"
+    rpy="-1.570796 0 -1.570796" />
+    <xacro:fixed_joint name="grasping_frame_joint"
+    parent="STS3215_03a-v1-4"
+    child="grasping_frame"
+    xyz="-0.02 -0.09 -0.03"
+    rpy="0 0 0" />
+  <!-- ======================== ACTUATED JOINTS ======================== -->
   <!-- Continuous Joints (Actuated) -->
   <xacro:revolute_joint name="joint1"
